Commit message: Enhance cargo_bot package with kinematic movement, configuration files, and RViz launch support

File: robotics_playground_ws/src/cargo_bot/urdf/cargo_bot.urdf.xacro (robot description, xacro)
@@ -5,6 +5,7 @@
   <xacro:include filename="$(find cargo_bot)/urdf/cargo_bot_base.xacro" />
   <xacro:include filename="$(find cargo_bot)/urdf/cargo_bot_wheels.xacro" />
+  <xacro:property name="geometry" value="${xacro.load_yaml('$(find cargo_bot)/config/cargo_bot_geometry.yaml')}" />
   <xacro:cargo_bot_materials visual_mode="$(arg visual_mode)" />
-  <xacro:cargo_bot_base />
-  <xacro:cargo_bot_wheels />
+  <xacro:cargo_bot_base geometry="${geometry}" />
+  <xacro:cargo_bot_wheels geometry="${geometry}" />
 </robot>

File: robotics_playground_ws/src/cargo_bot/urdf/cargo_bot_base.xacro (robot description, xacro)
@@ -1,14 +1,14 @@
 <?xml version="1.0"?>
 <robot xmlns:xacro="http://www.ros.org/wiki/xacro">
-  <xacro:macro name="cargo_bot_base">
-    <link name="base_footprint" />
+  <xacro:macro name="cargo_bot_base" params="geometry">
+    <link name="${geometry.frames.base_footprint}" />
     <joint name="base_footprint_joint" type="fixed">
-      <parent link="base_footprint" />
-      <child link="base_link" />
-      <origin xyz="0 0 0.23" rpy="0 0 0" />
+      <parent link="${geometry.frames.base_footprint}" />
+      <child link="${geometry.frames.base_link}" />
+      <origin xyz="0 0 ${geometry.base.base_link_z}" rpy="0 0 0" />
     </joint>
-    <link name="base_link" />
+    <link name="${geometry.frames.base_link}" />
     <joint name="chassis_joint" type="fixed">
-      <parent link="base_link" />
+      <parent link="${geometry.frames.base_link}" />
       <child link="chassis_link" />
       <origin xyz="0 0 0" rpy="0 0 0" />
@@ -18,5 +18,5 @@
         <origin xyz="0 0 0" rpy="0 0 0" />
         <geometry>
-          <box size="1.65 1.0 0.28" />
+          <box size="${geometry.chassis.length} ${geometry.chassis.width} ${geometry.chassis.height}" />
         </geometry>
         <material name="chassis_dark" />
@@ -24,7 +24,7 @@
     </link>
     <joint name="cargo_deck_joint" type="fixed">
-      <parent link="base_link" />
+      <parent link="${geometry.frames.base_link}" />
       <child link="cargo_deck_link" />
-      <origin xyz="-0.33 0 0.165" rpy="0 0 0" />
+      <origin xyz="${geometry.cargo_deck.x} ${geometry.cargo_deck.y} ${geometry.cargo_deck.z}" rpy="0 0 0" />
     </joint>
     <link name="cargo_deck_link">
@@ -32,5 +32,5 @@
         <origin xyz="0 0 0" rpy="0 0 0" />
         <geometry>
-          <box size="0.92 0.82 0.05" />
+          <box size="${geometry.cargo_deck.length} ${geometry.cargo_deck.width} ${geometry.cargo_deck.height}" />
         </geometry>
         <material name="cargo_deck_blue" />

File: robotics_playground_ws/src/cargo_bot/urdf/cargo_bot_wheels.xacro (robot description, xacro)
@@ -1,59 +1,59 @@
 <?xml version="1.0"?>
 <robot xmlns:xacro="http://www.ros.org/wiki/xacro">
-  <xacro:macro name="cargo_bot_wheels">
-    <joint name="left_wheel_joint" type="continuous">
-      <parent link="base_link" />
-      <child link="left_wheel_link" />
-      <origin xyz="0.32 0.58 0" rpy="0 0 0" />
+  <xacro:macro name="cargo_bot_wheels" params="geometry">
+    <joint name="${geometry.drive_wheels.left_joint}" type="continuous">
+      <parent link="${geometry.frames.base_link}" />
+      <child link="${geometry.drive_wheels.left_link}" />
+      <origin xyz="${geometry.drive_wheels.x} ${geometry.drive_wheels.y_offset} ${geometry.drive_wheels.z}" rpy="0 0 0" />
       <axis xyz="0 1 0" />
     </joint>
-    <link name="left_wheel_link">
+    <link name="${geometry.drive_wheels.left_link}">
       <visual>
         <origin xyz="0 0 0" rpy="1.57079632679 0 0" />
         <geometry>
-          <cylinder radius="0.23" length="0.14" />
+          <cylinder radius="${geometry.drive_wheels.radius}" length="${geometry.drive_wheels.width}" />
         </geometry>
         <material name="tire_black" />
       </visual>
       <visual>
-        <origin xyz="0 0.081 0" rpy="1.57079632679 0 0" />
+        <origin xyz="0 ${geometry.drive_wheels.hub_y_offset} 0" rpy="1.57079632679 0 0" />
         <geometry>
-          <cylinder radius="0.12" length="0.02" />
+          <cylinder radius="${geometry.drive_wheels.hub_radius}" length="${geometry.drive_wheels.hub_width}" />
         </geometry>
         <material name="safety_yellow" />
       </visual>
     </link>
-    <joint name="right_wheel_joint" type="continuous">
-      <parent link="base_link" />
-      <child link="right_wheel_link" />
-      <origin xyz="0.32 -0.58 0" rpy="0 0 0" />
+    <joint name="${geometry.drive_wheels.right_joint}" type="continuous">
+      <parent link="${geometry.frames.base_link}" />
+      <child link="${geometry.drive_wheels.right_link}" />
+      <origin xyz="${geometry.drive_wheels.x} ${-geometry.drive_wheels.y_offset} ${geometry.drive_wheels.z}" rpy="0 0 0" />
       <axis xyz="0 1 0" />
     </joint>
-    <link name="right_wheel_link">
+    <link name="${geometry.drive_wheels.right_link}">
       <visual>
         <origin xyz="0 0 0" rpy="1.57079632679 0 0" />
         <geometry>
-          <cylinder radius="0.23" length="0.14" />
+          <cylinder radius="${geometry.drive_wheels.radius}" length="${geometry.drive_wheels.width}" />
         </geometry>
         <material name="tire_black" />
       </visual>
       <visual>
-        <origin xyz="0 -0.081 0" rpy="1.57079632679 0 0" />
+        <origin xyz="0 ${-geometry.drive_wheels.hub_y_offset} 0" rpy="1.57079632679 0 0" />
         <geometry>
-          <cylinder radius="0.12" length="0.02" />
+          <cylinder radius="${geometry.drive_wheels.hub_radius}" length="${geometry.drive_wheels.hub_width}" />
         </geometry>
         <material name="safety_yellow" />
       </visual>
     </link>
-    <joint name="rear_support_wheel_joint" type="fixed">
-      <parent link="base_link" />
-      <child link="rear_support_wheel_link" />
-      <origin xyz="-0.62 0 -0.145" rpy="0 0 0" />
+    <joint name="${geometry.rear_support.joint}" type="fixed">
+      <parent link="${geometry.frames.base_link}" />
+      <child link="${geometry.rear_support.link}" />
+      <origin xyz="${geometry.rear_support.x} ${geometry.rear_support.y} ${geometry.rear_support.z}" rpy="0 0 0" />
     </joint>
-    <link name="rear_support_wheel_link">
+    <link name="${geometry.rear_support.link}">
       <visual>
         <origin xyz="0 0 0" rpy="0 0 0" />
         <geometry>
-          <sphere radius="0.085" />
+          <sphere radius="${geometry.rear_support.radius}" />
         </geometry>
         <material name="tire_black" />
