Commit message: Add manipulator model and update cargo_bot configuration and materials

File: robotics_playground_ws/src/cargo_bot/urdf/cargo_bot.urdf.xacro (robot description, xacro)
@@ -5,7 +5,9 @@
   <xacro:include filename="$(find cargo_bot)/urdf/cargo_bot_base.xacro" />
   <xacro:include filename="$(find cargo_bot)/urdf/cargo_bot_wheels.xacro" />
+  <xacro:include filename="$(find cargo_bot)/urdf/cargo_bot_manipulator.xacro" />
   <xacro:property name="geometry" value="${xacro.load_yaml('$(find cargo_bot)/config/cargo_bot_geometry.yaml')}" />
   <xacro:cargo_bot_materials visual_mode="$(arg visual_mode)" />
   <xacro:cargo_bot_base geometry="${geometry}" />
   <xacro:cargo_bot_wheels geometry="${geometry}" />
+  <xacro:cargo_bot_manipulator geometry="${geometry}" />
 </robot>

File: robotics_playground_ws/src/cargo_bot/urdf/cargo_bot_materials.xacro (robot description, xacro)
@@ -15,4 +15,13 @@
         <color rgba="1.0 0.68 0.12 0.55" />
       </material>
+      <material name="manipulator_steel">
+        <color rgba="0.62 0.68 0.74 0.65" />
+      </material>
+      <material name="manipulator_accent">
+        <color rgba="0.95 0.45 0.12 0.65" />
+      </material>
+      <material name="camera_black">
+        <color rgba="0.05 0.06 0.07 0.7" />
+      </material>
     </xacro:if>
     <xacro:unless value="${visual_mode == 'dev'}">
@@ -29,4 +38,13 @@
         <color rgba="1.0 0.68 0.12 1.0" />
       </material>
+      <material name="manipulator_steel">
+        <color rgba="0.62 0.68 0.74 1.0" />
+      </material>
+      <material name="manipulator_accent">
+        <color rgba="0.95 0.45 0.12 1.0" />
+      </material>
+      <material name="camera_black">
+        <color rgba="0.05 0.06 0.07 1.0" />
+      </material>
     </xacro:unless>
   </xacro:macro>

Commit message: Add collision and inertial properties for cargo_bot model in preparation for Gazebo simulation

File: robotics_playground_ws/src/cargo_bot/urdf/cargo_bot.urdf.xacro (robot description, xacro)
@@ -2,4 +2,5 @@
 <robot xmlns:xacro="http://www.ros.org/wiki/xacro" name="cargo_bot">
   <xacro:arg name="visual_mode" default="dev" />
+  <xacro:include filename="$(find cargo_bot)/urdf/cargo_bot_inertial.xacro" />
   <xacro:include filename="$(find cargo_bot)/urdf/cargo_bot_materials.xacro" />
   <xacro:include filename="$(find cargo_bot)/urdf/cargo_bot_base.xacro" />

File: robotics_playground_ws/src/cargo_bot/urdf/cargo_bot_base.xacro (robot description, xacro)
@@ -15,4 +15,9 @@
     </joint>
     <link name="chassis_link">
+      <xacro:box_inertial
+        mass="${geometry.chassis.mass}"
+        length="${geometry.chassis.length}"
+        width="${geometry.chassis.width}"
+        height="${geometry.chassis.height}" />
       <visual>
         <origin xyz="0 0 0" rpy="0 0 0" />
@@ -22,4 +27,10 @@
         <material name="chassis_dark" />
       </visual>
+      <collision>
+        <origin xyz="0 0 0" rpy="0 0 0" />
+        <geometry>
+          <box size="${geometry.chassis.length} ${geometry.chassis.width} ${geometry.chassis.height}" />
+        </geometry>
+      </collision>
     </link>
     <joint name="cargo_deck_joint" type="fixed">
@@ -29,4 +40,9 @@
     </joint>
     <link name="cargo_deck_link">
+      <xacro:box_inertial
+        mass="${geometry.cargo_deck.mass}"
+        length="${geometry.cargo_deck.length}"
+        width="${geometry.cargo_deck.width}"
+        height="${geometry.cargo_deck.height}" />
       <visual>
         <origin xyz="0 0 0" rpy="0 0 0" />
@@ -36,4 +52,10 @@
         <material name="cargo_deck_blue" />
       </visual>
+      <collision>
+        <origin xyz="0 0 0" rpy="0 0 0" />
+        <geometry>
+          <box size="${geometry.cargo_deck.length} ${geometry.cargo_deck.width} ${geometry.cargo_deck.height}" />
+        </geometry>
+      </collision>
     </link>
   </xacro:macro>

File: robotics_playground_ws/src/cargo_bot/urdf/cargo_bot_manipulator.xacro (robot description, xacro)
@@ -10,4 +10,8 @@
     </joint>
     <link name="${geometry.manipulator.mount.link}">
+      <xacro:cylinder_inertial
+        mass="${geometry.manipulator.mount.mass}"
+        radius="${geometry.manipulator.mount.radius}"
+        length="${geometry.manipulator.mount.height}" />
       <visual>
         <origin xyz="0 0 0" rpy="0 0 0" />
@@ -17,4 +21,10 @@
         <material name="manipulator_accent" />
       </visual>
+      <collision>
+        <origin xyz="0 0 0" rpy="0 0 0" />
+        <geometry>
+          <cylinder radius="${geometry.manipulator.mount.radius}" length="${geometry.manipulator.mount.height}" />
+        </geometry>
+      </collision>
     </link>
     <joint name="${geometry.manipulator.column.joint}" type="fixed">
@@ -24,4 +34,9 @@
     </joint>
     <link name="${geometry.manipulator.column.link}">
+      <xacro:box_inertial
+        mass="${geometry.manipulator.column.mass}"
+        length="${geometry.manipulator.column.length}"
+        width="${geometry.manipulator.column.width}"
+        height="${geometry.manipulator.column.height}" />
       <visual>
         <origin xyz="0 0 0" rpy="0 0 0" />
@@ -31,4 +46,10 @@
         <material name="manipulator_steel" />
       </visual>
+      <collision>
+        <origin xyz="0 0 0" rpy="0 0 0" />
+        <geometry>
+          <box size="${geometry.manipulator.column.length} ${geometry.manipulator.column.width} ${geometry.manipulator.column.height}" />
+        </geometry>
+      </collision>
     </link>
     <joint name="${geometry.manipulator.lift.joint}" type="prismatic">
@@ -40,4 +61,9 @@
     </joint>
     <link name="${geometry.manipulator.lift.link}">
+      <xacro:box_inertial
+        mass="${geometry.manipulator.lift.mass}"
+        length="${geometry.manipulator.lift.length}"
+        width="${geometry.manipulator.lift.width}"
+        height="${geometry.manipulator.lift.height}" />
       <visual>
         <origin xyz="0 0 0" rpy="0 0 0" />
@@ -47,4 +73,10 @@
         <material name="manipulator_accent" />
       </visual>
+      <collision>
+        <origin xyz="0 0 0" rpy="0 0 0" />
+        <geometry>
+          <box size="${geometry.manipulator.lift.length} ${geometry.manipulator.lift.width} ${geometry.manipulator.lift.height}" />
+        </geometry>
+      </collision>
     </link>
     <joint name="${geometry.manipulator.arm.housing.joint}" type="fixed">
@@ -54,4 +86,10 @@
     </joint>
     <link name="${geometry.manipulator.arm.housing.link}">
+      <xacro:box_inertial
+        mass="${geometry.manipulator.arm.housing.mass}"
+        length="${geometry.manipulator.arm.housing.length}"
+        width="${geometry.manipulator.arm.housing.width}"
+        height="${geometry.manipulator.arm.housing.height}"
+        origin_xyz="${geometry.manipulator.arm.housing.length / 2.0} 0 0" />
       <visual>
         <origin xyz="${geometry.manipulator.arm.housing.length / 2.0} 0 0" rpy="0 0 0" />
@@ -61,4 +99,10 @@
         <material name="manipulator_accent" />
       </visual>
+      <collision>
+        <origin xyz="${geometry.manipulator.arm.housing.length / 2.0} 0 0" rpy="0 0 0" />
+        <geometry>
+          <box size="${geometry.manipulator.arm.housing.length} ${geometry.manipulator.arm.housing.width} ${geometry.manipulator.arm.housing.height}" />
+        </geometry>
+      </collision>
     </link>
     <joint name="${geometry.manipulator.arm.extension.joint}" type="prismatic">
@@ -70,4 +114,10 @@
     </joint>
     <link name="${geometry.manipulator.arm.extension.link}">
+      <xacro:box_inertial
+        mass="${geometry.manipulator.arm.extension.mass}"
+        length="${geometry.manipulator.arm.extension.length}"
+        width="${geometry.manipulator.arm.extension.width}"
+        height="${geometry.manipulator.arm.extension.height}"
+        origin_xyz="${geometry.manipulator.arm.extension.length / 2.0} 0 0" />
       <visual>
         <origin xyz="${geometry.manipulator.arm.extension.length / 2.0} 0 0" rpy="0 0 0" />
@@ -77,4 +127,10 @@
         <material name="manipulator_steel" />
       </visual>
+      <collision>
+        <origin xyz="${geometry.manipulator.arm.extension.length / 2.0} 0 0" rpy="0 0 0" />
+        <geometry>
+          <box size="${geometry.manipulator.arm.extension.length} ${geometry.manipulator.arm.extension.width} ${geometry.manipulator.arm.extension.height}" />
+        </geometry>
+      </collision>
     </link>
     <joint name="${geometry.manipulator.gripper.base.joint}" type="fixed">
@@ -84,4 +140,10 @@
     </joint>
     <link name="${geometry.manipulator.gripper.base.link}">
+      <xacro:box_inertial
+        mass="${geometry.manipulator.gripper.base.mass}"
+        length="${geometry.manipulator.gripper.base.length}"
+        width="${geometry.manipulator.gripper.base.width}"
+        height="${geometry.manipulator.gripper.base.height}"
+        origin_xyz="${geometry.manipulator.gripper.base.length / 2.0} 0 0" />
       <visual>
         <origin xyz="${geometry.manipulator.gripper.base.length / 2.0} 0 0" rpy="0 0 0" />
@@ -91,4 +153,10 @@
         <material name="manipulator_accent" />
       </visual>
+      <collision>
+        <origin xyz="${geometry.manipulator.gripper.base.length / 2.0} 0 0" rpy="0 0 0" />
+        <geometry>
+          <box size="${geometry.manipulator.gripper.base.length} ${geometry.manipulator.gripper.base.width} ${geometry.manipulator.gripper.base.height}" />
+        </geometry>
+      </collision>
     </link>
     <joint name="${geometry.manipulator.gripper.fingers.left_joint}" type="prismatic">
@@ -100,4 +168,10 @@
     </joint>
     <link name="${geometry.manipulator.gripper.fingers.left_link}">
+      <xacro:box_inertial
+        mass="${geometry.manipulator.gripper.fingers.mass}"
+        length="${geometry.manipulator.gripper.fingers.length}"
+        width="${geometry.manipulator.gripper.fingers.width}"
+        height="${geometry.manipulator.gripper.fingers.height}"
+        origin_xyz="${geometry.manipulator.gripper.fingers.length / 2.0} 0 0" />
       <visual>
         <origin xyz="${geometry.manipulator.gripper.fingers.length / 2.0} 0 0" rpy="0 0 0" />
@@ -107,4 +181,10 @@
         <material name="safety_yellow" />
       </visual>
+      <collision>
+        <origin xyz="${geometry.manipulator.gripper.fingers.length / 2.0} 0 0" rpy="0 0 0" />
+        <geometry>
+          <box size="${geometry.manipulator.gripper.fingers.length} ${geometry.manipulator.gripper.fingers.width} ${geometry.manipulator.gripper.fingers.height}" />
+        </geometry>
+      </collision>
     </link>
     <joint name="${geometry.manipulator.gripper.fingers.right_joint}" type="prismatic">
@@ -117,4 +197,10 @@
     </joint>
     <link name="${geometry.manipulator.gripper.fingers.right_link}">
+      <xacro:box_inertial
+        mass="${geometry.manipulator.gripper.fingers.mass}"
+        length="${geometry.manipulator.gripper.fingers.length}"
+        width="${geometry.manipulator.gripper.fingers.width}"
+        height="${geometry.manipulator.gripper.fingers.height}"
+        origin_xyz="${geometry.manipulator.gripper.fingers.length / 2.0} 0 0" />
       <visual>
         <origin xyz="${geometry.manipulator.gripper.fingers.length / 2.0} 0 0" rpy="0 0 0" />
@@ -124,4 +210,10 @@
         <material name="safety_yellow" />
       </visual>
+      <collision>
+        <origin xyz="${geometry.manipulator.gripper.fingers.length / 2.0} 0 0" rpy="0 0 0" />
+        <geometry>
+          <box size="${geometry.manipulator.gripper.fingers.length} ${geometry.manipulator.gripper.fingers.width} ${geometry.manipulator.gripper.fingers.height}" />
+        </geometry>
+      </collision>
     </link>
     <joint name="${geometry.manipulator.gripper.camera.joint}" type="fixed">
@@ -131,4 +223,10 @@
     </joint>
     <link name="${geometry.manipulator.gripper.camera.link}">
+      <xacro:box_inertial
+        mass="${geometry.manipulator.gripper.camera.mass}"
+        length="${geometry.manipulator.gripper.camera.length}"
+        width="${geometry.manipulator.gripper.camera.width}"
+        height="${geometry.manipulator.gripper.camera.height}"
+        origin_xyz="${geometry.manipulator.gripper.camera.length / 2.0} 0 0" />
       <visual>
         <origin xyz="${geometry.manipulator.gripper.camera.bracket_x} 0 ${-geometry.manipulator.gripper.camera.bracket_z}" rpy="0 0 0" />
@@ -145,4 +243,10 @@
         <material name="camera_black" />
       </visual>
+      <collision>
+        <origin xyz="${geometry.manipulator.gripper.camera.length / 2.0} 0 0" rpy="0 0 0" />
+        <geometry>
+          <box size="${geometry.manipulator.gripper.camera.length} ${geometry.manipulator.gripper.camera.width} ${geometry.manipulator.gripper.camera.height}" />
+        </geometry>
+      </collision>
     </link>
   </xacro:macro>

File: robotics_playground_ws/src/cargo_bot/urdf/cargo_bot_wheels.xacro (robot description, xacro)
@@ -9,4 +9,9 @@
     </joint>
     <link name="${geometry.drive_wheels.left_link}">
+      <xacro:cylinder_inertial
+        mass="${geometry.drive_wheels.mass}"
+        radius="${geometry.drive_wheels.radius}"
+        length="${geometry.drive_wheels.width}"
+        origin_rpy="1.57079632679 0 0" />
       <visual>
         <origin xyz="0 0 0" rpy="1.57079632679 0 0" />
@@ -16,4 +21,10 @@
         <material name="tire_black" />
       </visual>
+      <collision>
+        <origin xyz="0 0 0" rpy="1.57079632679 0 0" />
+        <geometry>
+          <cylinder radius="${geometry.drive_wheels.radius}" length="${geometry.drive_wheels.width}" />
+        </geometry>
+      </collision>
       <visual>
         <origin xyz="0 ${geometry.drive_wheels.hub_y_offset} 0" rpy="1.57079632679 0 0" />
@@ -31,4 +42,9 @@
     </joint>
     <link name="${geometry.drive_wheels.right_link}">
+      <xacro:cylinder_inertial
+        mass="${geometry.drive_wheels.mass}"
+        radius="${geometry.drive_wheels.radius}"
+        length="${geometry.drive_wheels.width}"
+        origin_rpy="1.57079632679 0 0" />
       <visual>
         <origin xyz="0 0 0" rpy="1.57079632679 0 0" />
@@ -38,4 +54,10 @@
         <material name="tire_black" />
       </visual>
+      <collision>
+        <origin xyz="0 0 0" rpy="1.57079632679 0 0" />
+        <geometry>
+          <cylinder radius="${geometry.drive_wheels.radius}" length="${geometry.drive_wheels.width}" />
+        </geometry>
+      </collision>
       <visual>
         <origin xyz="0 ${-geometry.drive_wheels.hub_y_offset} 0" rpy="1.57079632679 0 0" />
@@ -52,4 +74,7 @@
     </joint>
     <link name="${geometry.rear_support.link}">
+      <xacro:sphere_inertial
+        mass="${geometry.rear_support.mass}"
+        radius="${geometry.rear_support.radius}" />
       <visual>
         <origin xyz="0 0 0" rpy="0 0 0" />
@@ -59,4 +84,10 @@
         <material name="tire_black" />
       </visual>
+      <collision>
+        <origin xyz="0 0 0" rpy="0 0 0" />
+        <geometry>
+          <sphere radius="${geometry.rear_support.radius}" />
+        </geometry>
+      </collision>
     </link>
   </xacro:macro>

Commit message: Add sensor integration and testing for cargo bot simulation
- Introduced new sensor materials in cargo_bot_materials.xacro for better visualization.
- Created cargo_bot_sensors.xacro to define LIDAR and IMU sensors with appropriate configurations.
- Updated cargo_bot_wheels.xacro to include a joint state publisher plugin for better state management.
- Enhanced gazebo_warehouse.launch.py and indoor_rooms.launch.py to support multiple sensor configurations and profiles.
- Implemented realistic and ideal sensor tests in test_launch_gazebo_realistic_localization.py and test_launch_indoor_ideal.py to validate sensor performance.
- Added new test cases in test_launch_gazebo_warehouse.py to ensure proper functioning of the robot in the Gazebo environment.
- Updated indoor_rooms.sdf and small_warehouse.sdf to include necessary sensor plugins for simulation.

File: robotics_playground_ws/src/cargo_bot/urdf/cargo_bot.urdf.xacro (robot description, xacro)
@@ -7,8 +7,11 @@
   <xacro:include filename="$(find cargo_bot)/urdf/cargo_bot_wheels.xacro" />
   <xacro:include filename="$(find cargo_bot)/urdf/cargo_bot_manipulator.xacro" />
+  <xacro:include filename="$(find cargo_bot)/urdf/cargo_bot_sensors.xacro" />
   <xacro:property name="geometry" value="${xacro.load_yaml('$(find cargo_bot)/config/cargo_bot_geometry.yaml')}" />
+  <xacro:property name="sensor_config" value="${xacro.load_yaml('$(find cargo_bot)/config/sensors.yaml')}" />
   <xacro:cargo_bot_materials visual_mode="$(arg visual_mode)" />
   <xacro:cargo_bot_base geometry="${geometry}" />
   <xacro:cargo_bot_wheels geometry="${geometry}" />
   <xacro:cargo_bot_manipulator geometry="${geometry}" />
+  <xacro:cargo_bot_sensors geometry="${geometry}" sensor_config="${sensor_config}" />
 </robot>

File: robotics_playground_ws/src/cargo_bot/urdf/cargo_bot_materials.xacro (robot description, xacro)
@@ -24,4 +24,7 @@
         <color rgba="0.05 0.06 0.07 0.7" />
       </material>
+      <material name="sensor_black">
+        <color rgba="0.02 0.03 0.04 0.7" />
+      </material>
     </xacro:if>
     <xacro:unless value="${visual_mode == 'dev'}">
@@ -47,4 +50,7 @@
         <color rgba="0.05 0.06 0.07 1.0" />
       </material>
+      <material name="sensor_black">
+        <color rgba="0.02 0.03 0.04 1.0" />
+      </material>
     </xacro:unless>
   </xacro:macro>

File: robotics_playground_ws/src/cargo_bot/urdf/cargo_bot_wheels.xacro (robot description, xacro)
@@ -100,9 +100,15 @@
         <topic>/cmd_vel</topic>
         <odom_topic>/odom</odom_topic>
-        <tf_topic>/tf</tf_topic>
+        <tf_topic>/ground_truth/tf</tf_topic>
         <frame_id>odom</frame_id>
         <child_frame_id>${geometry.frames.base_footprint}</child_frame_id>
         <odom_publish_frequency>50</odom_publish_frequency>
       </plugin>
+      <plugin filename="gz-sim-joint-state-publisher-system"
+              name="gz::sim::systems::JointStatePublisher">
+        <topic>/sim/joint_states</topic>
+        <joint_name>${geometry.drive_wheels.left_joint}</joint_name>
+        <joint_name>${geometry.drive_wheels.right_joint}</joint_name>
+      </plugin>
     </gazebo>
   </xacro:macro>
