Commit message: Add initial implementation of cargo_bot_world package with warehouse model
- Created model configuration and SDF files for aws_robomaker_warehouse_WallB_01.
- Added package.xml and setup.py for package management and dependencies.
- Included test files for copyright, flake8, and PEP257 compliance.
- Defined small_warehouse world with various models and lighting configurations.

File: robotics_playground_ws/src/cargo_bot/urdf/cargo_bot_manipulator.xacro (robot description, xacro)
@@ -8,4 +8,5 @@
       <axis xyz="0 0 1" />
       <limit lower="${geometry.manipulator.mount.lower}" upper="${geometry.manipulator.mount.upper}" effort="${geometry.manipulator.mount.effort}" velocity="${geometry.manipulator.mount.velocity}" />
+      <dynamics damping="500" friction="100"/>
     </joint>
     <link name="${geometry.manipulator.mount.link}">
@@ -59,4 +60,5 @@
       <axis xyz="0 0 1" />
       <limit lower="${geometry.manipulator.lift.lower}" upper="${geometry.manipulator.lift.upper}" effort="${geometry.manipulator.lift.effort}" velocity="${geometry.manipulator.lift.velocity}" />
+      <dynamics damping="500" friction="100"/>
     </joint>
     <link name="${geometry.manipulator.lift.link}">
@@ -112,4 +114,5 @@
       <axis xyz="1 0 0" />
       <limit lower="${geometry.manipulator.arm.extension.lower}" upper="${geometry.manipulator.arm.extension.upper}" effort="${geometry.manipulator.arm.extension.effort}" velocity="${geometry.manipulator.arm.extension.velocity}" />
+      <dynamics damping="500" friction="100"/>
     </joint>
     <link name="${geometry.manipulator.arm.extension.link}">
@@ -166,4 +169,5 @@
       <axis xyz="0 1 0" />
       <limit lower="${geometry.manipulator.gripper.fingers.lower}" upper="${geometry.manipulator.gripper.fingers.upper}" effort="${geometry.manipulator.gripper.fingers.effort}" velocity="${geometry.manipulator.gripper.fingers.velocity}" />
+      <dynamics damping="100" friction="20"/>
     </joint>
     <link name="${geometry.manipulator.gripper.fingers.left_link}">

File: robotics_playground_ws/src/cargo_bot/urdf/cargo_bot_wheels.xacro (robot description, xacro)
@@ -91,4 +91,19 @@
       </collision>
     </link>
+    <gazebo>
+      <plugin filename="gz-sim-diff-drive-system"
+              name="gz::sim::systems::DiffDrive">
+        <left_joint>${geometry.drive_wheels.left_joint}</left_joint>
+        <right_joint>${geometry.drive_wheels.right_joint}</right_joint>
+        <wheel_separation>${2 * geometry.drive_wheels.y_offset}</wheel_separation>
+        <wheel_radius>${geometry.drive_wheels.radius}</wheel_radius>
+        <topic>/cmd_vel</topic>
+        <odom_topic>/odom</odom_topic>
+        <tf_topic>/tf</tf_topic>
+        <frame_id>odom</frame_id>
+        <child_frame_id>${geometry.frames.base_footprint}</child_frame_id>
+        <odom_publish_frequency>50</odom_publish_frequency>
+      </plugin>
+    </gazebo>
   </xacro:macro>
 </robot>
