Commit message: Add unit and acceptance tests for navigation and collision detection
- Implement unit tests for navigation cancellation responses in `test_goal_navigator.py`.
- Enhance SLAM mapping tests in `test_launch_slam_mapping.py` by adding IMU data handling.
- Create acceptance tests for static navigation in `test_launch_static_navigation.py` and long navigation scenarios in `test_launch_static_navigation_long.py`.
- Add tests for corridor-to-room navigation turns in `test_launch_static_navigation_turn.py`.
- Introduce tests for occupancy-grid collision checks in `test_map_collision.py`.
- Update path planning configuration tests in `test_path_planning_config.py` to reflect new parameters.
- Modify SLAM configuration tests in `test_slam_config.py` for updated mapping parameters.
- Establish static navigation configuration tests in `test_static_navigation_config.py` to ensure trajectory execution contracts are met.
- Update indoor room launch file to include manipulator state publishing for complete TF branch connectivity in RViz.

File: robotics_playground_ws/src/cargo_bot/urdf/cargo_bot_base.xacro (robot description, xacro)
@@ -9,4 +9,12 @@
     </joint>
     <link name="${geometry.frames.base_link}" />
+    <!-- Nav2 control point: midpoint of the differential-drive axle. The
+         physical model and saved map remain anchored at base_footprint. -->
+    <joint name="base_axle_joint" type="fixed">
+      <parent link="${geometry.frames.base_footprint}" />
+      <child link="${geometry.frames.base_axle}" />
+      <origin xyz="${geometry.drive_wheels.x} 0 0" rpy="0 0 0" />
+    </joint>
+    <link name="${geometry.frames.base_axle}" />
     <joint name="chassis_joint" type="fixed">
       <parent link="${geometry.frames.base_link}" />
@@ -19,5 +27,7 @@
         length="${geometry.chassis.length}"
         width="${geometry.chassis.width}"
-        height="${geometry.chassis.height}" />
+        height="${geometry.chassis.height}"
+        origin_xyz="0 0 ${geometry.chassis.inertial_z}"
+        roll_pitch_multiplier="${geometry.chassis.roll_pitch_inertia_multiplier}" />
       <visual>
         <origin xyz="0 0 0" rpy="0 0 0" />

File: robotics_playground_ws/src/cargo_bot/urdf/cargo_bot_inertial.xacro (robot description, xacro)
@@ -1,13 +1,13 @@
 <?xml version="1.0"?>
 <robot xmlns:xacro="http://www.ros.org/wiki/xacro">
-  <xacro:macro name="box_inertial" params="mass length width height origin_xyz:='0 0 0'">
+  <xacro:macro name="box_inertial" params="mass length width height origin_xyz:='0 0 0' roll_pitch_multiplier:=1.0">
     <inertial>
       <origin xyz="${origin_xyz}" rpy="0 0 0" />
       <mass value="${mass}" />
       <inertia
-        ixx="${(mass / 12.0) * ((width * width) + (height * height))}"
+        ixx="${roll_pitch_multiplier * (mass / 12.0) * ((width * width) + (height * height))}"
         ixy="0"
         ixz="0"
-        iyy="${(mass / 12.0) * ((length * length) + (height * height))}"
+        iyy="${roll_pitch_multiplier * (mass / 12.0) * ((length * length) + (height * height))}"
         iyz="0"
         izz="${(mass / 12.0) * ((length * length) + (width * width))}" />

File: robotics_playground_ws/src/cargo_bot/urdf/cargo_bot_manipulator.xacro (robot description, xacro)
@@ -5,5 +5,6 @@
       <parent link="${geometry.frames.base_link}" />
       <child link="${geometry.manipulator.mount.link}" />
-      <origin xyz="${geometry.manipulator.mount.x} ${geometry.manipulator.mount.y} ${geometry.manipulator.mount.z}" rpy="0 0 0" />
+      <!-- The safe transport/home pose points the complete manipulator behind the base. -->
+      <origin xyz="${geometry.manipulator.mount.x} ${geometry.manipulator.mount.y} ${geometry.manipulator.mount.z}" rpy="0 0 3.14159265359" />
       <axis xyz="0 0 1" />
       <limit lower="${geometry.manipulator.mount.lower}" upper="${geometry.manipulator.mount.upper}" effort="${geometry.manipulator.mount.effort}" velocity="${geometry.manipulator.mount.velocity}" />

File: robotics_playground_ws/src/cargo_bot/urdf/cargo_bot_wheels.xacro (robot description, xacro)
@@ -91,4 +91,10 @@
       </collision>
     </link>
+    <!-- Near-ideal profile: model the rear ball as a freely sliding support,
+         rather than a third rubber contact that resists differential turns. -->
+    <gazebo reference="${geometry.rear_support.link}">
+      <mu1>0.001</mu1>
+      <mu2>0.001</mu2>
+    </gazebo>
     <gazebo>
       <plugin filename="gz-sim-diff-drive-system"
@@ -98,4 +104,8 @@
         <wheel_separation>${2 * geometry.drive_wheels.y_offset}</wheel_separation>
         <wheel_radius>${geometry.drive_wheels.radius}</wheel_radius>
+        <max_linear_acceleration>${geometry.drive_wheels.controller.max_linear_acceleration}</max_linear_acceleration>
+        <min_linear_acceleration>${geometry.drive_wheels.controller.min_linear_acceleration}</min_linear_acceleration>
+        <max_angular_acceleration>${geometry.drive_wheels.controller.max_angular_acceleration}</max_angular_acceleration>
+        <min_angular_acceleration>${geometry.drive_wheels.controller.min_angular_acceleration}</min_angular_acceleration>
         <topic>/cmd_vel</topic>
         <odom_topic>/wheel_model/odometry</odom_topic>
